File: Schematics/Final Project Schematic/MHDP.sch (KiCad schematic (older format))
At the start: 62 parts, among them Q0 PN2222A, Q1 PN2222A, Q2 PN2222A, Q3 PN2222A, SW0 Slow Down, SW1 Play/Pause, SW2 Speed Up, U0 ATMEGA328P-PU, U1 BA70BC0T, U2 LM7805_TO220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

Commit message: Update Schematic + BOM
Parts:
- removed POT0: POT, symbol R
- added J0: Programmer Header, symbol Conn_02x03_Counter_Clockwise
- added RV0: POT, symbol POT
- RS0: value 1 -> 1K
Connections:
- net +3.3V: now also J0.3 (Pin_3)
- net AUDIO: now also Q?.2 (B), J0.6 (Pin_6); no longer RS0.2
- net GND: now also RS0.2, J0.1 (Pin_1)
- net RST: now reaches R9.2, U0.1 ((PCINT14/~RESET~)PC6)
- net RST: now also J0.4 (Pin_4)
- net SCK: now reaches DP0.1 (K), U0.19 ((PCINT5/SCK)PB5)
- net SCK: now also J0.5 (Pin_5)
- net at RS0.1: no longer Q?.2 (B)
- net at RS1.2: now also RV0.1
- net at LS0.2: now also RV0.2
- net PULSE0 renamed MOSI
- net MOSI: now also J0.2 (Pin_2)
- no-connect marks 0 -> 1
Other:
- note added: "Programmer Header"
Changed lines of the file:
@@
-$EndComp
-$Comp
-L R RS0
-U 1 1 5FB79ADD
-P 5400 4150
-F 0 "RS0" V 5480 4150 50  0000 C CNN
-F 1 "1" V 5400 4150 50  0000 C CNN
-F 2 "" V 5330 4150 50  0001 C CNN
-F 3 "" H 5400 4150 50  0001 C CNN
-	1    5400 4150
-	0    1    1    0
-$EndComp
-$Comp
-L R POT0
-U 1 1 5FB7A30A
-P 6450 3850
-F 0 "POT0" V 6530 3850 50  0000 C CNN
-F 1 "POT" V 6450 3850 50  0000 C CNN
-F 2 "" V 6380 3850 50  0001 C CNN
-F 3 "" H 6450 3850 50  0001 C CNN
-	1    6450 3850
-	0    1    1    0
 $EndComp
 $Comp
@@
 Text Notes 5200 4050 0    60   ~ 0
 Sound\nControl\nModule
-Text Label 4000 4150 0    60   ~ 0
+Text Label 4500 4100 0    60   ~ 0
 AUDIO
 Wire Wire Line
@@
 	5850 3850 6050 3850
 Wire Wire Line
+	6150 3650 6150 4000
+Wire Wire Line
+	6050 3850 6050 3650
+Wire Notes Line
+	5200 4550 6850 4550
+Wire Notes Line
+	6850 4550 6850 3750
+Wire Notes Line
+	6850 3750 5200 3750
+Wire Notes Line
+	5200 3750 5200 4550
+Wire Wire Line
+	4800 4150 5550 4150
+Wire Wire Line
+	4800 4150 4800 4100
+Wire Wire Line
+	4800 4100 4450 4100
+Wire Wire Line
+	4450 4100 4450 4150
+$Comp
+L R RS0
+U 1 1 5FB8F39C
+P 5400 4300
+F 0 "RS0" V 5480 4300 50  0000 C CNN
+F 1 "1K" V 5400 4300 50  0000 C CNN
+F 2 "" V 5330 4300 50  0001 C CNN
+F 3 "" H 5400 4300 50  0001 C CNN
+	1    5400 4300
+	1    0    0    -1
+$EndComp
+$Comp
+L GND #PWR?
+U 1 1 5FB8FCE1
+P 5400 4450
+F 0 "#PWR?" H 5400 4200 50  0001 C CNN
+F 1 "GND" H 5400 4300 50  0000 C CNN
+F 2 "" H 5400 4450 50  0001 C CNN
+F 3 "" H 5400 4450 50  0001 C CNN
+	1    5400 4450
+	0    -1   -1   0
+$EndComp
+$Comp
+L Conn_02x03_Counter_Clockwise J0
+U 1 1 5FB988B2
+P 4300 3650
+F 0 "J0" H 4350 3850 50  0000 C CNN
+F 1 "Programmer Header" H 4350 3450 50  0000 C CNN
+F 2 "" H 4300 3650 50  0001 C CNN
+F 3 "" H 4300 3650 50  0001 C CNN
+	1    4300 3650
+	1    0    0    -1
+$EndComp
+Wire Wire Line
+	3800 3550 4100 3550
+$Comp
+L GND #PWR?
+U 1 1 5FB9D618
+P 3800 3550
+F 0 "#PWR?" H 3800 3300 50  0001 C CNN
+F 1 "GND" H 3800 3400 50  0000 C CNN
+F 2 "" H 3800 3550 50  0001 C CNN
+F 3 "" H 3800 3550 50  0001 C CNN
+	1    3800 3550
+	0    1    1    0
+$EndComp
+Wire Wire Line
+	4100 3650 3800 3650
+Text Label 3800 3650 0    60   ~ 0
+MOSI
+Text Label 3550 4050 0    60   ~ 0
+MOSI
+Wire Wire Line
+	3550 4050 3050 4050
+Wire Wire Line
+	4100 3750 3800 3750
+Text Label 3800 3750 0    60   ~ 0
++3.3V
+Text Label 4700 3550 0    60   ~ 0
+MISO
+Wire Wire Line
+	4600 3550 4700 3550
+Wire Wire Line
+	4600 3650 4700 3650
+Wire Wire Line
+	4600 3750 4700 3750
+Wire Wire Line
+	4450 4150 3050 4150
+Text Label 3550 4150 0    60   ~ 0
+MISO
+Text Label 4700 3650 0    60   ~ 0
+SCK
+Text Label 3550 4250 0    60   ~ 0
+SCK
+Text Label 4700 3750 0    60   ~ 0
+RST
+Text Label 3550 5200 0    60   ~ 0
+RST
+Text Notes 4050 3400 0    60   ~ 0
+Programmer Header
+Wire Notes Line
+	3600 3300 5000 3300
+Wire Notes Line
+	5000 3300 5000 3900
+Wire Notes Line
+	5000 3900 3600 3900
+Wire Notes Line
+	3600 3900 3600 3300
+$Comp
+L POT RV0
+U 1 1 5FBAF02A
+P 6450 3850
+F 0 "RV0" V 6275 3850 50  0000 C CNN
+F 1 "POT" V 6350 3850 50  0000 C CNN
+F 2 "" H 6450 3850 50  0001 C CNN
+F 3 "" H 6450 3850 50  0001 C CNN
+	1    6450 3850
+	0    1    1    0
+$EndComp
+Wire Wire Line
+	6650 3850 6650 3900
+Wire Wire Line
 	6600 3850 6650 3850
 Wire Wire Line
-	6650 3850 6650 3900
-Wire Wire Line
-	6150 3850 6300 3850
-Wire Wire Line
-	6150 3650 6150 3850
-Wire Wire Line
-	6050 3850 6050 3650
-Wire Notes Line
-	5200 4550 6850 4550
-Wire Notes Line
-	6850 4550 6850 3750
-Wire Notes Line
-	6850 3750 5200 3750
-Wire Notes Line
-	5200 3750 5200 4550
-Wire Wire Line
-	5250 4150 4800 4150
-Wire Wire Line
-	4800 4150 4800 4100
-Wire Wire Line
-	4800 4100 4450 4100
-Wire Wire Line
-	4450 4150 4450 4100
-Wire Wire Line
-	3050 4150 4450 4150
+	6150 4000 6450 4000
+NoConn ~ 6300 3850
 $EndSCHEMATC

Commit message: Update Schematic + BOM
Parts:
- added D4: LED, symbol LED
- added PD3: D_Photo, symbol D_Photo
- added Q4: PN2222A, TO_SOT_Packages_THT:TO-92_Molded_Narrow, symbol PN2222A
- added RD4: 1K, symbol R
Connections:
- net +3.3V: now also D4.2 (A), PD3.2 (A), Q4.3 (C)
- net GND: now also RD4.2
- net DATAV: now reaches U0.27 ((PCINT12/SDA/ADC4)PC4)
- net DATAV: now also Q4.1 (E), RD4.1
- net at D0.1 (K), D1.1 (K), D2.1 (K)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: now also D4.1 (K)
- new net: PD3.1 (K), Q4.2 (B)
Other:
- moved on the sheet: D0, D1, D2, D3, DM0, DM1, DM2, DM3, DM4, DM5, DM6, DM7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

Commit message: Update schematic labels for motor pin colors
Other:
- note added: "Black"
- note added: "Yellow"
Changed lines of the file:
@@
 Wire Notes Line
 	8050 3100 8050 500
+Text Notes 5150 2300 0    60   ~ 0
+Yellow
+Text Notes 5150 2000 0    60   ~ 0
+Black
 $EndSCHEMATC

Commit message: Update schematic
Parts:
- added D5: D, symbol D
- added SW3: Power Switch, symbol SW_Push
Connections:
- net +7V: now also D5.2 (A)
- net at C0.1, C2.1, C4.1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: now also D5.1 (K), SW3.2; no longer BT0.1 (+)
- new net: BT0.1 (+), SW3.1
Other:
- moved on the sheet: BT0
Changed lines of the file:
@@
 L Battery BT0
 U 1 1 5FB42C0E
-P 750 900
-F 0 "BT0" H 850 1000 50  0000 L CNN
-F 1 "9V" H 850 900 50  0000 L CNN
-F 2 "" V 750 960 50  0001 C CNN
-F 3 "" V 750 960 50  0001 C CNN
-	1    750  900
-	-1   0    0    1
+P 1050 750
+F 0 "BT0" H 1150 850 50  0000 L CNN
+F 1 "9V" H 1150 750 50  0000 L CNN
+F 2 "" V 1050 810 50  0001 C CNN
+F 3 "" V 1050 810 50  0001 C CNN
+	1    1050 750
+	0    -1   -1   0
 $EndComp
 $Comp
 L GND #PWR?
 U 1 1 5FB42D1E
-P 750 700
-F 0 "#PWR?" H 750 450 50  0001 C CNN
-F 1 "GND" H 750 550 50  0000 C CNN
-F 2 "" H 750 700 50  0001 C CNN
-F 3 "" H 750 700 50  0001 C CNN
-	1    750  700
-	-1   0    0    1
+P 1250 750
+F 0 "#PWR?" H 1250 500 50  0001 C CNN
+F 1 "GND" H 1250 600 50  0000 C CNN
+F 2 "" H 1250 750 50  0001 C CNN
+F 3 "" H 1250 750 50  0001 C CNN
+	1    1250 750
+	0    -1   -1   0
 $EndComp
 $Comp
@@
 Wire Wire Line
 	1650 1200 1650 1150
-Connection ~ 750  1850
-Wire Wire Line
-	750  1850 1000 1850
-Wire Wire Line
-	750  2550 1000 2550
-Connection ~ 750  1150
+Wire Wire Line
+	650  1850 1000 1850
+Wire Wire Line
+	650  2550 1000 2550
 Connection ~ 950  1150
 Wire Wire Line
-	950  1150 950  1200
-Wire Wire Line
-	750  1150 1000 1150
-Wire Wire Line
-	750  1100 750  2550
+	950  900  950  1200
+Wire Wire Line
+	650  1150 1000 1150
 Wire Wire Line
 	4800 1900 5100 1900
@@
 Text Notes 5150 2000 0    60   ~ 0
 Black
+$Comp
+L SW_Push SW3
+U 1 1 5FBFFF54
+P 650 950
+F 0 "SW3" H 700 1050 50  0000 L CNN
+F 1 "Power Switch" H 650 890 50  0000 C CNN
+F 2 "" H 650 1150 50  0001 C CNN
+F 3 "" H 650 1150 50  0001 C CNN
+	1    650  950
+	0    1    1    0
+$EndComp
+Wire Wire Line
+	650  750  850  750
+Wire Wire Line
+	650  1150 650  2550
+Connection ~ 650  1850
+$Comp
+L D D5
+U 1 1 5FC0512F
+P 1250 900
+F 0 "D5" H 1250 1000 50  0000 C CNN
+F 1 "D" H 1250 800 50  0000 C CNN
+F 2 "" H 1250 900 50  0001 C CNN
+F 3 "" H 1250 900 50  0001 C CNN
+	1    1250 900
+	1    0    0    -1
+$EndComp
+Wire Wire Line
+	1750 1150 1750 900
+Wire Wire Line
+	1750 900  1400 900
+Connection ~ 1750 1150
+Wire Wire Line
+	1100 900  950  900
 $EndSCHEMATC
